Commit message: geting rviz to work

File: catkin_ws/src/my_robot/urdf/my_robot.xacro (robot description, xacro)
@@ -1,4 +1,19 @@
 <?xml version='1.0'?>
 <robot name="my_robot" xmlns:xacro="http://www.ros.org/wiki/xacro">
+  <material name="blue">
+    <color rgba="0 0 1 1"/>
+  </material>
+  <material name="green">
+    <color rgba="0 1 0 1"/>
+  </material>
+  <material name="grey">
+    <color rgba="0.7 0.7 0.7 1"/>
+  </material>
+  <material name="red">
+    <color rgba="1 0 0 1"/>
+  </material>
+  <material name="black">
+    <color rgba="0 0 0 1"/>
+  </material>
   <xacro:include filename="$(find my_robot)/urdf/my_robot.gazebo" />
   <link name="robot_footprint"></link>
@@ -172,5 +187,5 @@
       <origin xyz="0 0 0" rpy="0 0 0"/>
       <geometry>
-        <mesh filename="model://hokuyo/meshes/hokuyo.dae"/>
+        <mesh filename="package://my_robot/meshes/hokuyo.dae"/>
       </geometry>
       <material name="black"/>

Commit message: changing robot desgin

File: catkin_ws/src/my_robot/urdf/my_robot.xacro (robot description, xacro)
@@ -15,4 +15,13 @@
   <material name="black">
     <color rgba="0 0 0 1"/>
+  </material>
+  <material name="yellow">
+    <color rgba="1 1 0 1"/>
+  </material>
+  <material name="white">
+    <color rgba="1 1 1 1"/>
+  </material>
+  <material name="top_cylinder_blue_material">
+    <color rgba="0 0 1 1"/>
   </material>
   <xacro:include filename="$(find my_robot)/urdf/my_robot.gazebo" />
@@ -24,5 +33,5 @@
   </joint>
   <link name='chassis'>
-    <pose>0 0 0.1 0 0 0</pose>
+    <pose>0 0 0.06 0 0 0</pose>
     <inertial>
       <mass value="15.0"/>
@@ -37,37 +46,44 @@
       <origin xyz="0 0 0" rpy="0 0 0"/>
       <geometry>
-        <box size=".4 .2 .1"/>
-      </geometry>
-    </collision>
-    <visual name='chassis_visual'>
-      <origin xyz="0 0 0" rpy="0 0 0"/>
-      <geometry>
-        <box size=".4 .2 .1"/>
-      </geometry>
-      <material name="blue"/>
+        <box size=".45 .33 .06"/>
+      </geometry>
+    </collision>
+    <visual name='chassis_visual_base'>
+      <origin xyz="0 0 0" rpy="0 0 0"/>
+      <geometry>
+        <box size=".45 .33 .06"/>
+      </geometry>
+      <material name="yellow"/>
+    </visual>
+    <visual name='chassis_visual_top'>
+      <origin xyz="0 0 0.03" rpy="0 0 0"/>
+      <geometry>
+        <cylinder radius="0.08" length="0.05"/>
+      </geometry>
+      <material name="top_cylinder_blue_material"/>
     </visual>
     <collision name='back_caster_collision'>
-      <origin xyz="-0.15 0 -0.05" rpy="0 0 0"/>
-      <geometry>
-        <sphere radius="0.0499"/>
+      <origin xyz="-0.15 0 -0.06" rpy="0 0 0"/>
+      <geometry>
+        <sphere radius="0.035"/>
       </geometry>
     </collision>
     <visual name='back_caster_visual'>
-      <origin xyz="-0.15 0 -0.05" rpy="0 0 0"/>
-      <geometry>
-        <sphere radius="0.05"/>
+      <origin xyz="-0.15 0 -0.06" rpy="0 0 0"/>
+      <geometry>
+        <sphere radius="0.035"/>
       </geometry>
       <material name="grey"/>
     </visual>
     <collision name='front_caster_collision'>
-      <origin xyz="0.15 0 -0.05" rpy="0 0 0"/>
-      <geometry>
-        <sphere radius="0.0499"/>
+      <origin xyz="0.15 0 -0.06" rpy="0 0 0"/>
+      <geometry>
+        <sphere radius="0.035"/>
       </geometry>
     </collision>
     <visual name='front_caster_visual'>
-      <origin xyz="0.15 0 -0.05" rpy="0 0 0"/>
-      <geometry>
-        <sphere radius="0.05"/>
+      <origin xyz="0.15 0 -0.06" rpy="0 0 0"/>
+      <geometry>
+        <sphere radius="0.035"/>
       </geometry>
       <material name="grey"/>
@@ -87,11 +103,11 @@
       <origin xyz="0 0 0" rpy="0 1.5707 1.5707"/>
       <geometry>
-        <cylinder radius="0.1" length="0.05"/>
-      </geometry>
-    </collision>
-    <visual>
-      <origin xyz="0 0 0" rpy="0 1.5707 1.5707"/>
-      <geometry>
-        <cylinder radius="0.1" length="0.05"/>
+        <cylinder radius="0.10" length="0.025"/>
+      </geometry>
+    </collision>
+    <visual>
+      <origin xyz="0 0 0" rpy="0 1.5707 1.5707"/>
+      <geometry>
+        <cylinder radius="0.10" length="0.025"/>
       </geometry>
       <material name="green"/>
@@ -111,11 +127,11 @@
       <origin xyz="0 0 0" rpy="0 1.5707 1.5707"/>
       <geometry>
-        <cylinder radius="0.1" length="0.05"/>
-      </geometry>
-    </collision>
-    <visual>
-      <origin xyz="0 0 0" rpy="0 1.5707 1.5707"/>
-      <geometry>
-        <cylinder radius="0.1" length="0.05"/>
+        <cylinder radius="0.10" length="0.025"/>
+      </geometry>
+    </collision>
+    <visual>
+      <origin xyz="0 0 0" rpy="0 1.5707 1.5707"/>
+      <geometry>
+        <cylinder radius="0.10" length="0.025"/>
       </geometry>
       <material name="green"/>
@@ -123,5 +139,5 @@
   </link>
   <joint type="continuous" name="left_wheel_joint">
-    <origin xyz="0 0.15 0" rpy="0 0 0"/>
+    <origin xyz="0 0.165 0" rpy="0 0 0"/>
     <child link="left_wheel"/>
     <parent link="chassis"/>
@@ -131,5 +147,5 @@
   </joint>
   <joint type="continuous" name="right_wheel_joint">
-    <origin xyz="0 -0.15 0" rpy="0 0 0"/>
+    <origin xyz="0 -0.165 0" rpy="0 0 0"/>
     <child link="right_wheel"/>
     <parent link="chassis"/>
@@ -193,12 +209,13 @@
   </link>
   <joint name="hokuyo_joint" type="fixed">
-    <origin xyz="0.15 0 0.1" rpy="0 0 0"/>
+    <origin xyz="0.15 0 0.08" rpy="0 0 0"/>
     <parent link="chassis"/>
     <child link="hokuyo"/>
     <axis xyz="0 1 0"/>
   </joint>
-  <!-- GAZEBO REFERENCES FOR MATERIALS -->
-  <!-- These tags tell Gazebo how to apply the defined URDF materials -->
   <gazebo reference="chassis">
+    <material>Gazebo/Yellow</material>
+  </gazebo>
+  <gazebo reference="chassis_visual_top">
     <material>Gazebo/Blue</material>
   </gazebo>

Commit message: review fixes

File: catkin_ws/src/my_robot/urdf/my_robot.xacro (robot description, xacro)
@@ -56,38 +56,60 @@
       <material name="yellow"/>
     </visual>
-    <visual name='chassis_visual_top'>
-      <origin xyz="0 0 0.03" rpy="0 0 0"/>
+    <collision name='back_caster_collision'>
+      <origin xyz="-0.15 0 -0.025" rpy="0 0 0"/>
+      <geometry>
+        <sphere radius="0.035"/>
+      </geometry>
+    </collision>
+    <visual name='back_caster_visual'>
+      <origin xyz="-0.15 0 -0.025" rpy="0 0 0"/>
+      <geometry>
+        <sphere radius="0.035"/>
+      </geometry>
+      <material name="grey"/>
+    </visual>
+    <collision name='front_caster_collision'>
+      <origin xyz="0.15 0 -0.025" rpy="0 0 0"/>
+      <geometry>
+        <sphere radius="0.035"/>
+      </geometry>
+    </collision>
+    <visual name='front_caster_visual'>
+      <origin xyz="0.15 0 -0.025" rpy="0 0 0"/>
+      <geometry>
+        <sphere radius="0.035"/>
+      </geometry>
+      <material name="grey"/>
+    </visual>
+  </link>
+  <link name='top_cylinder_link'>
+    <inertial>
+      <mass value="0.1"/>
+      <origin xyz="0 0 0" rpy="0 0 0"/>
+      <inertia
+        ixx="1e-6" ixy="0" ixz="0"
+        iyy="1e-6" iyz="0"
+        izz="1e-6"
+      />
+    </inertial>
+    <collision>
+      <origin xyz="0 0 0" rpy="0 0 0"/>
       <geometry>
         <cylinder radius="0.08" length="0.05"/>
       </geometry>
+    </collision>
+    <visual>
+      <origin xyz="0 0 0" rpy="0 0 0"/>
+      <geometry>
+        <cylinder radius="0.08" length="0.05"/>
+      </geometry>
       <material name="top_cylinder_blue_material"/>
     </visual>
-    <collision name='back_caster_collision'>
-      <origin xyz="-0.15 0 -0.06" rpy="0 0 0"/>
-      <geometry>
-        <sphere radius="0.035"/>
-      </geometry>
-    </collision>
-    <visual name='back_caster_visual'>
-      <origin xyz="-0.15 0 -0.06" rpy="0 0 0"/>
-      <geometry>
-        <sphere radius="0.035"/>
-      </geometry>
-      <material name="grey"/>
-    </visual>
-    <collision name='front_caster_collision'>
-      <origin xyz="0.15 0 -0.06" rpy="0 0 0"/>
-      <geometry>
-        <sphere radius="0.035"/>
-      </geometry>
-    </collision>
-    <visual name='front_caster_visual'>
-      <origin xyz="0.15 0 -0.06" rpy="0 0 0"/>
-      <geometry>
-        <sphere radius="0.035"/>
-      </geometry>
-      <material name="grey"/>
-    </visual>
-  </link>
+  </link>
+  <joint name="top_cylinder_joint" type="fixed">
+    <origin xyz="0 0 0.055" rpy="0 0 0"/>
+    <parent link="chassis"/>
+    <child link="top_cylinder_link"/>
+  </joint>
   <link name='left_wheel'>
     <inertial>
@@ -103,11 +125,11 @@
       <origin xyz="0 0 0" rpy="0 1.5707 1.5707"/>
       <geometry>
-        <cylinder radius="0.10" length="0.025"/>
-      </geometry>
-    </collision>
-    <visual>
-      <origin xyz="0 0 0" rpy="0 1.5707 1.5707"/>
-      <geometry>
-        <cylinder radius="0.10" length="0.025"/>
+        <cylinder radius="0.08" length="0.025"/>
+      </geometry>
+    </collision>
+    <visual>
+      <origin xyz="0 0 0" rpy="0 1.5707 1.5707"/>
+      <geometry>
+        <cylinder radius="0.08" length="0.025"/>
       </geometry>
       <material name="green"/>
@@ -127,11 +149,11 @@
       <origin xyz="0 0 0" rpy="0 1.5707 1.5707"/>
       <geometry>
-        <cylinder radius="0.10" length="0.025"/>
-      </geometry>
-    </collision>
-    <visual>
-      <origin xyz="0 0 0" rpy="0 1.5707 1.5707"/>
-      <geometry>
-        <cylinder radius="0.10" length="0.025"/>
+        <cylinder radius="0.08" length="0.025"/>
+      </geometry>
+    </collision>
+    <visual>
+      <origin xyz="0 0 0" rpy="0 1.5707 1.5707"/>
+      <geometry>
+        <cylinder radius="0.08" length="0.025"/>
       </geometry>
       <material name="green"/>
@@ -139,5 +161,5 @@
   </link>
   <joint type="continuous" name="left_wheel_joint">
-    <origin xyz="0 0.165 0" rpy="0 0 0"/>
+    <origin xyz="0 0.165 0.02" rpy="0 0 0"/>
     <child link="left_wheel"/>
     <parent link="chassis"/>
@@ -147,5 +169,5 @@
   </joint>
   <joint type="continuous" name="right_wheel_joint">
-    <origin xyz="0 -0.165 0" rpy="0 0 0"/>
+    <origin xyz="0 -0.165 0.02" rpy="0 0 0"/>
     <child link="right_wheel"/>
     <parent link="chassis"/>
@@ -167,11 +189,11 @@
       <origin xyz="0 0 0" rpy="0 0 0"/>
       <geometry>
-        <box size="0.05 0.05 0.05"/>
-      </geometry>
-    </collision>
-    <visual>
-      <origin xyz="0 0 0" rpy="0 0 0"/>
-      <geometry>
-        <box size="0.05 0.05 0.05"/>
+        <box size="0.06 0.06 0.06"/>
+      </geometry>
+    </collision>
+    <visual>
+      <origin xyz="0 0 0" rpy="0 0 0"/>
+      <geometry>
+        <box size="0.06 0.06 0.06"/>
       </geometry>
       <material name="red"/>
@@ -179,5 +201,5 @@
   </link>
   <joint name="camera_joint" type="fixed">
-    <origin xyz="0.2 0 0" rpy="0 0 0"/>
+    <origin xyz="0.225 0 0.03" rpy="0 0 0"/>
     <parent link="chassis"/>
     <child link="camera"/>
@@ -209,5 +231,5 @@
   </link>
   <joint name="hokuyo_joint" type="fixed">
-    <origin xyz="0.15 0 0.08" rpy="0 0 0"/>
+    <origin xyz="0.15 0 0.085" rpy="0 0 0"/>
     <parent link="chassis"/>
     <child link="hokuyo"/>
@@ -217,5 +239,5 @@
     <material>Gazebo/Yellow</material>
   </gazebo>
-  <gazebo reference="chassis_visual_top">
+  <gazebo reference="top_cylinder_link">
     <material>Gazebo/Blue</material>
   </gazebo>
